Commit message: Fixed some errors

File: catkin_ws/src/my_robot/urdf/my_bot.xacro (robot description, xacro)
@@ -80,7 +80,7 @@
     	iyy="0.1" iyz="0"
    	izz="0.1"
-      />z="0.1"
+      />
     </inertial>
-    <collision name='collision'>
+    <collision>
       <origin xyz="0 0 0" rpy=" 0 1.5707 1.5707"/>
       <geometry>
@@ -88,5 +88,5 @@
       </geometry>
     </collision>
-    <visual name='visual'>
+    <visual>
       <origin xyz="0 0 0" rpy=" 0 1.5707 1.5707"/>
       <geometry>
@@ -103,7 +103,7 @@
     	iyy="0.1" iyz="0"
    	izz="0.1"
-      />z="0.1"
+      />
     </inertial>
-    <collision name='collision'>
+    <collision>
       <origin xyz="0 0 0" rpy=" 0 1.5707 1.5707"/>
       <geometry>
@@ -111,5 +111,5 @@
       </geometry>
     </collision>
-    <visual name='visual'>
+    <visual>
       <origin xyz="0 0 0" rpy=" 0 1.5707 1.5707"/>
       <geometry>
